Commit message: change of shoulder frame

File: data/robots/dual_arm_iiwa7.urdf.xacro (robot description, xacro)
@@ -11,8 +11,8 @@
   <!--iiwa-->
   <xacro:iiwa7 hardware_interface="$(arg hardware_interface)" robot_name="left_arm" parent="world">
-    <origin xyz="0.2 0 0.0" rpy="0 0 0" />
+    <origin xyz="0.225 0 0.0" rpy="0 1.5708 0" />
   </xacro:iiwa7>
   <xacro:iiwa7 hardware_interface="$(arg hardware_interface)" robot_name="right_arm" parent="world">
-    <origin xyz="-0.2 0 0.0" rpy="0 0 0" />
+    <origin xyz="-0.225 0 0.0" rpy="0 -1.5708 0" />
   </xacro:iiwa7>
 </robot>

Commit message: Changed values to make arm plugs face same direction. Tweaked distance between arms.

File: data/robots/dual_arm_iiwa7.urdf.xacro (robot description, xacro)
@@ -11,8 +11,8 @@
   <!--iiwa-->
   <xacro:iiwa7 hardware_interface="$(arg hardware_interface)" robot_name="left_arm" parent="world">
-    <origin xyz="0.225 0 0.0" rpy="0 1.5708 0" />
+    <origin xyz="0.065 0 0" rpy="1.5708 0 1.5708" />
   </xacro:iiwa7>
   <xacro:iiwa7 hardware_interface="$(arg hardware_interface)" robot_name="right_arm" parent="world">
-    <origin xyz="-0.225 0 0.0" rpy="0 -1.5708 0" />
+    <origin xyz="-0.065 0 0" rpy="-1.5708 0 1.5708" />
   </xacro:iiwa7>
 </robot>
