Commit message: Added xacro and mesh files for dual-arm torso and Baxter pedestal.

File: data/robots/dual_arm_robot.xacro (robot description, xacro)
@@ -3,49 +3,20 @@
     <xacro:arg name="robot_name" default="dual_arm"/>
     <xacro:arg name="hardware_interface" default="PositionJointInterface"/>
+    <!-- pedestal -->
+    <xacro:include filename="$(find arm_ordata)/data/robots/baxter_pedestal.xacro"/>
+    <xacro:baxter_pedestal robot_name="$(arg robot_name)"/>
+    <!-- torso -->
+    <xacro:include filename="$(find arm_ordata)/data/robots/dual_arm_torso.xacro"/>
+    <xacro:dual_arm_torso robot_name="$(arg robot_name)" parent="$(arg robot_name)_base_plate_mount"/>
+    <!-- iiwa arms -->
     <!-- Import Rviz colors -->
-    <xacro:include filename="$(find iiwa_description)/urdf/materials.xacro" />
+    <xacro:include filename="$(find iiwa_description)/urdf/materials.xacro"/>
     <!--Import the lbr iiwa macro -->
     <xacro:include filename="$(find iiwa_description)/urdf/iiwa7.xacro"/>
-    <material name="LightGrey">
-        <color rgba="0.7 0.7 0.7 1"/>
-    </material>
-    <!--<xacro:macro name="iiwa7" params="robot_name hardware_interface robot_name">-->
-        <link name="$(arg robot_name)_base_plate">
-            <visual>
-                <origin xyz="0 0 0" rpy="0 0 0"/>
-                <geometry>
-                    <mesh filename="package://arm_ordata/data/robots/meshes/torso_visual_model.stl"/>
-                </geometry>
-                <material name="LightGrey"/>
-            </visual>
-            <collision>
-                <origin xyz="0 0 0" rpy="0 0 0"/>
-                <geometry>
-                    <mesh filename="package://arm_ordata/data/robots/meshes/torso_visual_model.stl"/>
-                </geometry>
-                <material name="LightGrey"/>
-            </collision>
-        </link>
-        <link name="$(arg robot_name)_left_arm_mount"/>
-        <link name="$(arg robot_name)_right_arm_mount"/>
-        <joint name="$(arg robot_name)_left_arm_mount_joint" type="fixed">
-            <parent link="$(arg robot_name)_base_plate"/>
-            <child link="$(arg robot_name)_left_arm_mount"/>
-            <origin xyz="-0.02 0.1384885 0.385" rpy="-1.5707963268 0 -0.785398163397448"/>
-            <axis xyz="0 0 1"/>
-        </joint>
-        <joint name="$(arg robot_name)_right_arm_mount_joint" type="fixed">
-            <parent link="$(arg robot_name)_base_plate"/>
-            <child link="$(arg robot_name)_right_arm_mount"/>
-            <origin xyz="-0.02 -0.1384885 0.385" rpy="1.5707963268 0 0.785398163397448"/>
-            <axis xyz="0 0 1"/>
-        </joint>
-        <!--iiwa-->
-        <xacro:iiwa7 hardware_interface="$(arg hardware_interface)" robot_name="$(arg robot_name)_left_arm" parent="$(arg robot_name)_left_arm_mount">
-            <origin xyz="0 0 0" rpy="0 0 0" />
-        </xacro:iiwa7>
-        <xacro:iiwa7 hardware_interface="$(arg hardware_interface)" robot_name="$(arg robot_name)_right_arm" parent="$(arg robot_name)_right_arm_mount">
-            <origin xyz="0 0 0" rpy="0 0 0" />
-        </xacro:iiwa7>
-    <!--</xacro:macro>-->
+    <xacro:iiwa7 hardware_interface="$(arg hardware_interface)" robot_name="$(arg robot_name)_left_arm" parent="$(arg robot_name)_left_arm_mount">
+        <origin xyz="0 0 0" rpy="0 0 0"/>
+    </xacro:iiwa7>
+    <xacro:iiwa7 hardware_interface="$(arg hardware_interface)" robot_name="$(arg robot_name)_right_arm" parent="$(arg robot_name)_right_arm_mount">
+        <origin xyz="0 0 0" rpy="0 0 0"/>
+    </xacro:iiwa7>
 </robot>
